Commit message: External package merged in
Still not working

File: line_follower_race_car/urdf/bicycle_bot.urdf.xacro (robot description, xacro)
@@ -12,5 +12,5 @@
 <robot name="bicycle_bot" xmlns:xacro="http://wiki.ros.org/xacro">
   <!-- Include xacro for inertials, materials and wheels -->
-  <xacro:include filename="$(find steer_bot_description)/urdf/wheel.xacro"/>
+  <xacro:include filename="$(find line_follower_race_car)/urdf/wheel.xacro"/>
   <xacro:property name="robot_namespace" value="/bicycle_bot"/>
   <!-- Gazebo plugins -->

File: line_follower_race_car/urdf/mogi_bot.xacro (robot description, xacro)
@@ -12,5 +12,5 @@
     wheel_separation_w = base_width  + 2 * axle_offset = 0.4
 -->
-<robot name="steer_bot" xmlns:xacro="http://wiki.ros.org/xacro">
+<robot name="mogi_bot" xmlns:xacro="http://wiki.ros.org/xacro">
   <!-- Include xacro for inertials, materials and wheels -->
   <xacro:include filename="$(find line_follower_race_car)/urdf/wheel.xacro"/>
@@ -23,5 +23,5 @@
       <robotNamespace>${robot_namespace}</robotNamespace>
       <robotSimType>steer_bot_hardware_gazebo/SteerBotHardwareGazebo</robotSimType>
-      <legacyModeNS>false</legacyModeNS>
+      <legacyModeNS>true</legacyModeNS>
     </plugin>
   </gazebo>
@@ -29,13 +29,13 @@
   <xacro:property name="deg_to_rad" value="0.01745329251994329577"/>
   <!-- Robot base dimensions -->
-  <xacro:property name="base_length" value="0.4" />
+  <xacro:property name="base_length" value="0.6" />
   <xacro:property name="base_width" value="0.2" />
   <xacro:property name="base_height" value="0.1" />
   <xacro:property name="base_mass" value="15" />
-  <xacro:property name="base_rpy" value="0 0 -1.5707"
+  <xacro:property name="base_rpy" value="0 0 0" />
   <!-- Wheel link dimensions -->
   <xacro:property name="wheel_radius" value="0.1" />
-  <xacro:property name="wheel_thickness" value="0.08" />
-  <xacro:property name="wheel_mass" value="1" />
+  <xacro:property name="wheel_thickness" value="0.05" />
+  <xacro:property name="wheel_mass" value="5" />
   <!-- Steering link dimensions -->
   <xacro:property name="steer_radius" value="0.05" />
@@ -45,8 +45,15 @@
   <xacro:property name="axle_offset" value="0.05" />
   <xacro:property name="steer_offset" value="0.02" />
+  <!-- Base footprint -->
+  <link name="base_footprint"></link>
+  <joint name="base_footprint_joint" type="fixed">
+    <origin xyz="0 0 0" rpy="0 0 -1.5707" />
+    <parent link="base_footprint"/>
+    <child link="base_link" />
+  </joint>
   <!-- Base link -->
   <link name="base_link">
     <visual>
-      <origin xyz="0 0 0" rpy="${base_rpy}"/>
+      <origin xyz="0 0 0" rpy="0 0 -1.5707"/>
       <geometry>
         <mesh filename = "package://line_follower_race_car/meshes/body.dae"/>
@@ -132,7 +139,7 @@
     <origin xyz="${-base_length/2+axle_offset} ${+base_width/2+axle_offset} 0" rpy="${-90 * deg_to_rad} 0 0"/>
   </xacro:rear_wheel_lr>
-  <!-- Colour -->
+  <!-- Colour
   <gazebo reference="base_link">
     <material>Gazebo/Green</material>
-  </gazebo>
+  </gazebo> -->
 </robot>

File: line_follower_race_car/urdf/wheel.xacro (robot description, xacro)
@@ -9,6 +9,6 @@
 <robot name="wheel" xmlns:xacro="http://wiki.ros.org/xacro">
   <!-- Include xacro for materials and inertials -->
-  <xacro:include filename="$(find racecar_description)/urdf/materials.xacro"/>
-  <xacro:include filename="$(find racecar_description)/urdf/inertials.xacro"/>
+  <xacro:include filename="$(find line_follower_race_car)/urdf/materials.xacro"/>
+  <xacro:include filename="$(find line_follower_race_car)/urdf/inertials.xacro"/>
   <!-- Properties -->
   <xacro:property name="steer_effort" value="10.0"/>
@@ -115,7 +115,7 @@
     <link name="${name}_wheel_link">
       <visual>
-        <origin xyz="0 0 0" rpy="0 0 0"/>
-        <geometry>
-          <cylinder radius="${wheel_radius}" length="${wheel_thickness}"/>
+        <origin xyz="0 0 0" rpy="0 1.5707 1.5707"/>
+        <geometry>
+          <mesh filename = "package://line_follower_race_car/meshes/front_wheels.dae"/>
         </geometry>
         <material name="red" />
@@ -124,5 +124,5 @@
         <origin xyz="0 0 0" rpy="0 1.5707 1.5707"/>
         <geometry>
-          <mesh filename = "package://line_follower_race_car/meshes/front_wheels.dae"/>
+          <cylinder radius="${wheel_radius}" length="${wheel_thickness}"/>
         </geometry>
       </collision>
@@ -135,6 +135,6 @@
       <parent link="${name}_steer_link"/>
       <child link="${name}_wheel_link"/>
-      <origin xyz="0 0 ${-steer_height}" rpy="${-90 * deg_to_rad} 0 0"/>
-      <axis xyz="0 0 1"/>
+      <origin xyz="0 0 ${-steer_height}" rpy="0 0 0"/>
+      <axis xyz="0 1 0"/>
     </joint>
     <transmission name="${name}_steer_joint_trans">
@@ -161,7 +161,8 @@
       <material>Gazebo/Blue</material>
     </gazebo>
+    <!--
     <gazebo reference="${name}_wheel_link">
       <material>Gazebo/Red</material>
-    </gazebo>
+    </gazebo> -->
   </xacro:macro>
   <!-- Bicycle model rear wheel link (required for steer_drive_controller) -->
@@ -267,7 +268,7 @@
         <origin xyz="0 0 0" rpy="0 0 0"/>
         <geometry>
-          <cylinder radius="${wheel_radius}" length="${wheel_thickness}"/>
-        </geometry>
-        <material name="red" />
+          <mesh filename = "package://line_follower_race_car/meshes/front_wheels.dae"/>
+        </geometry>
+        <!--<material name="red" />-->
       </visual>
       <collision>
@@ -298,7 +299,8 @@
       </joint>
     </transmission>
+    <!--
     <gazebo reference="${name}_wheel_link">
       <material>Gazebo/Red</material>
-    </gazebo>
+    </gazebo> -->
   </xacro:macro>
 </robot>
