Commit message: Lego race car

File: line_follower_race_car/urdf/mogi_bot.xacro (robot description, xacro)
@@ -1,20 +1,20 @@
 <?xml version='1.0'?>
 <robot name="mogi_bot" xmlns:xacro="http://www.ros.org/wiki/xacro">
-  <!-- Gazebo plugin -->
+  <!-- STEP 3 - Gazebo plugin -->
   <xacro:include filename="$(find line_follower_race_car)/urdf/mogi_bot.gazebo" />
-  <!-- RViz colors -->
+  <!-- STEP 4 - RViz colors -->
   <xacro:include filename="$(find line_follower_race_car)/urdf/materials.xacro" />
+  <!-- STEP 1 - Robot chassis -->
   <link name="base_footprint"></link>
   <joint name="base_footprint_joint" type="fixed">
-    <origin xyz="0 0 0" rpy="0 0 0" />
+    <origin xyz="0 0 0" rpy="0 0 -1.5707" />
     <parent link="base_footprint"/>
     <child link="base_link" />
   </joint>
-  <!-- Robot chassis -->
   <link name='base_link'>
     <pose>0 0 0.1 0 0 0</pose>
     <inertial>
       <mass value="15.0"/>
-      <origin xyz="0.0 0 0" rpy="0 0 0"/>
+      <origin xyz="0.0 0 0" rpy=" 0 0 0"/>
       <inertia
           ixx="0.1" ixy="0" ixz="0"
@@ -24,5 +24,5 @@
     </inertial>
     <collision name='collision'>
-      <origin xyz="0 0 0" rpy="0 0 0"/>
+      <origin xyz="0 0 0" rpy=" 0 0 -1.5707"/>
       <geometry>
         <box size=".4 .2 .1"/>
@@ -30,40 +30,16 @@
     </collision>
     <visual name='base_link_visual'>
-      <origin xyz="0 0 0" rpy="0 0 0"/>
+      <origin xyz="0 0 0" rpy=" 0 0 -1.5707"/>
       <geometry>
         <!--box size=".4 .2 .1"/-->
-        <mesh filename = "package://line_follower_race_car/meshes/mogi_bot.dae"/>
-      </geometry>
-      <material name="orange"/>
-    </visual>
-    <collision name='rear_caster_collision'>
-      <origin xyz="-0.15 0 -0.05" rpy="0 0 0"/>
-      <geometry>
-        <sphere radius="0.0499"/>
-      </geometry>
-    </collision>
-    <visual name='rear_caster_visual'>
-      <origin xyz="-0.15 0 -0.05" rpy="0 0 0"/>
-      <geometry>
-        <sphere radius="0.05"/>
-      </geometry>
-    </visual>
-    <collision name='front_caster_collision'>
-      <origin xyz="0.15 0 -0.05" rpy="0 0 0"/>
-      <geometry>
-        <sphere radius="0.0499"/>
-      </geometry>
-    </collision>
-    <visual name='front_caster_visual'>
-      <origin xyz="0.15 0 -0.05" rpy="0 0 0"/>
-      <geometry>
-        <sphere radius="0.05"/>
+        <mesh filename = "package://line_follower_race_car/meshes/body.dae"/>
       </geometry>
     </visual>
   </link>
-  <!-- Wheels -->
-  <joint type="continuous" name="left_wheel_joint">
-    <origin xyz="0 0.15 0" rpy="0 0 0"/>
-    <child link="left_wheel"/>
+  <!-- STEP 2 - Wheels -->
+  <!-- Front left -->
+  <joint type="continuous" name="front_left_wheel_joint">
+    <origin xyz="0.23 0.17 0" rpy="0 0 0"/>
+    <child link="front_left_wheel"/>
     <parent link="base_link"/>
     <axis xyz="0 1 0" rpy="0 0 0"/>
@@ -71,5 +47,5 @@
     <dynamics damping="1.0" friction="1.0"/>
   </joint>
-  <link name='left_wheel'>
+  <link name='front_left_wheel'>
     <inertial>
       <mass value="5.0"/>
@@ -87,16 +63,16 @@
       </geometry>
     </collision>
-    <visual name='left_wheel_visual'>
+    <visual name='front_left_wheel_visual'>
       <origin xyz="0 0 0" rpy="0 1.5707 1.5707"/>
       <geometry>
         <!--cylinder radius=".1" length=".05"/-->
-        <mesh filename = "package://line_follower_race_car/meshes/wheel.dae"/>
+        <mesh filename = "package://line_follower_race_car/meshes/front_wheels.dae"/>
       </geometry>
-      <material name="green"/>
     </visual>
   </link>
-  <joint type="continuous" name="right_wheel_joint">
-    <origin xyz="0 -0.15 0" rpy="0 0 0"/>
-    <child link="right_wheel"/>
+<!-- Front right -->
+  <joint type="continuous" name="front_right_wheel_joint">
+    <origin xyz="0.23 -0.19 0" rpy="0 0 0"/>
+    <child link="front_right_wheel"/>
     <parent link="base_link"/>
     <axis xyz="0 1 0" rpy="0 0 0"/>
@@ -104,5 +80,38 @@
     <dynamics damping="1.0" friction="1.0"/>
   </joint>
-  <link name='right_wheel'>
+  <link name='front_right_wheel'>
+    <inertial>
+      <mass value="5.0"/>
+      <origin xyz="0 0 0" rpy="0 1.5707 -1.5707"/>
+      <inertia
+          ixx="0.1" ixy="0" ixz="0"
+          iyy="0.1" iyz="0"
+          izz="0.1"
+      />
+    </inertial>
+    <collision name='collision'>
+      <origin xyz="0 0 0" rpy="0 1.5707 -1.5707"/>
+      <geometry>
+        <cylinder radius=".1" length=".05"/>
+      </geometry>
+    </collision>
+    <visual name='front_right_wheel_visual'>
+      <origin xyz="0 0 0" rpy="0 1.5707 -1.5707"/>
+      <geometry>
+        <!--cylinder radius=".1" length=".05"/-->
+        <mesh filename = "package://line_follower_race_car/meshes/front_wheels.dae"/>
+      </geometry>
+    </visual>
+  </link>
+<!-- Rear left -->
+  <joint type="continuous" name="rear_left_wheel_joint">
+    <origin xyz="-0.25 0.17 0" rpy="0 0 0"/>
+    <child link="rear_left_wheel"/>
+    <parent link="base_link"/>
+    <axis xyz="0 1 0" rpy="0 0 0"/>
+    <limit effort="10000" velocity="1000"/>
+    <dynamics damping="1.0" friction="1.0"/>
+  </joint>
+  <link name='rear_left_wheel'>
     <inertial>
       <mass value="5.0"/>
@@ -120,89 +129,42 @@
       </geometry>
     </collision>
-    <visual name='right_wheel_visual'>
+    <visual name='rear_left_wheel_visual'>
       <origin xyz="0 0 0" rpy="0 1.5707 1.5707"/>
       <geometry>
         <!--cylinder radius=".1" length=".05"/-->
-        <mesh filename = "package://line_follower_race_car/meshes/wheel.dae"/>
+        <mesh filename = "package://line_follower_race_car/meshes/front_wheels.dae"/>
       </geometry>
-      <material name="green"/>
     </visual>
   </link>
-    <!-- Camera -->
-  <joint type="fixed" name="camera_joint">
-    <origin xyz="0.225 0 0.075" rpy="0 0 0"/>
-    <child link="camera_link"/>
+<!-- Rear right -->
+  <joint type="continuous" name="rear_right_wheel_joint">
+    <origin xyz="-0.25 -0.19 0" rpy="0 0 0"/>
+    <child link="rear_right_wheel"/>
     <parent link="base_link"/>
-    <axis xyz="0 1 0" />
+    <axis xyz="0 1 0" rpy="0 0 0"/>
+    <limit effort="10000" velocity="1000"/>
+    <dynamics damping="1.0" friction="1.0"/>
   </joint>
-  <link name='camera_link'>
-    <pose>0 0 0 0 0 0</pose>
+  <link name='rear_right_wheel'>
     <inertial>
-      <mass value="0.1"/>
-      <origin xyz="0 0 0" rpy="0 0 0"/>
+      <mass value="5.0"/>
+      <origin xyz="0 0 0" rpy="0 1.5707 -1.5707"/>
       <inertia
-          ixx="1e-6" ixy="0" ixz="0"
-          iyy="1e-6" iyz="0"
-          izz="1e-6"
+          ixx="0.1" ixy="0" ixz="0"
+          iyy="0.1" iyz="0"
+          izz="0.1"
       />
     </inertial>
     <collision name='collision'>
-      <origin xyz="0 0 0" rpy="0 0 0"/>
+      <origin xyz="0 0 0" rpy="0 1.5707 -1.5707"/>
       <geometry>
-        <box size=".05 .05 .05"/>
+        <cylinder radius=".1" length=".05"/>
       </geometry>
     </collision>
-    <visual name='camera_link_visual'>
-      <origin xyz="0 0 0" rpy="0 0 0"/>
+    <visual name='rear_right_wheel_visual'>
+      <origin xyz="0 0 0" rpy="0 1.5707 -1.5707"/>
       <geometry>
-        <box size=".05 .05 .05"/>
-      </geometry>
-    </visual>
-  </link>
-  <gazebo reference="camera_link">
-    <material>Gazebo/Red</material>
-  </gazebo>
-  <joint type="fixed" name="camera_optical_joint">
-    <origin xyz="0 0 0" rpy="-1.5707 0 -1.5707"/>
-    <child link="camera_link_optical"/>
-    <parent link="camera_link"/>
-  </joint>
-  <link name="camera_link_optical">
-  </link>
-  <!-- IMU -->
-  <joint name="imu_joint" type="fixed">
-    <origin xyz="0 0 0" rpy="0 0 0" />
-    <parent link="base_link"/>
-    <child link="imu_link" />
-  </joint>
-  <link name="imu_link">
-  </link>
-  <!-- Lidar -->
-  <joint type="fixed" name="scan_joint">
-    <origin xyz="0.0 0 0.15" rpy="0 0 0"/>
-    <child link="scan_link"/>
-    <parent link="base_link"/>
-    <axis xyz="0 1 0" rpy="0 0 0"/>
-  </joint>
-  <link name='scan_link'>
-    <inertial>
-      <mass value="1e-5"/>
-      <origin xyz="0 0 0" rpy="0 0 0"/>
-      <inertia
-          ixx="1e-6" ixy="0" ixz="0"
-          iyy="1e-6" iyz="0"
-          izz="1e-6"
-      />
-    </inertial>
-    <collision name='collision'>
-      <origin xyz="0 0 0" rpy="0 0 0"/>
-      <geometry>
-        <box size=".1 .1 .1"/>
-      </geometry>
-    </collision>
-    <visual name='scan_link_visual'>
-      <origin xyz="0 0 0" rpy="0 0 0"/>
-      <geometry>
-        <mesh filename = "package://line_follower_race_car/meshes/lidar.dae"/>
+        <!--cylinder radius=".1" length=".05"/-->
+        <mesh filename = "package://line_follower_race_car/meshes/front_wheels.dae"/>
       </geometry>
     </visual>

Commit message: Kamera felszerelése

File: line_follower_race_car/urdf/mogi_bot.xacro (robot description, xacro)
@@ -170,3 +170,44 @@
     </visual>
   </link>
+    <!-- Camera -->
+  <joint type="fixed" name="camera_joint">
+    <origin xyz="0.300 -0.005 0.075" rpy="0 0 0"/>
+    <child link="camera_link"/>
+    <parent link="base_link"/>
+    <axis xyz="0 1 0" />
+  </joint>
+  <link name='camera_link'>
+    <pose>0 0 0 0 0 0</pose>
+    <inertial>
+      <mass value="0.1"/>
+      <origin xyz="0 0 0" rpy="0 0 0"/>
+      <inertia
+          ixx="1e-6" ixy="0" ixz="0"
+          iyy="1e-6" iyz="0"
+          izz="1e-6"
+      />
+    </inertial>
+    <collision name='collision'>
+      <origin xyz="0 0 0" rpy="0 0 0"/>
+      <geometry>
+        <box size=".05 .05 .05"/>
+      </geometry>
+    </collision>
+    <visual name='camera_link_visual'>
+      <origin xyz="0 0 0" rpy="0 0 0"/>
+      <geometry>
+        <box size=".05 .05 .05"/>
+      </geometry>
+    </visual>
+  </link>
+  <gazebo reference="camera_link">
+    <material>Gazebo/Red</material>
+  </gazebo>
+  <joint type="fixed" name="camera_optical_joint">
+    <origin xyz="0 0 0" rpy="-1.5707 0 -1.5707"/>
+    <child link="camera_link_optical"/>
+    <parent link="camera_link"/>
+  </joint>
+  <link name="camera_link_optical">
+  </link>
 </robot>

Commit message: Update mogi_bot.xacro

File: line_follower_race_car/urdf/mogi_bot.xacro (robot description, xacro)
@@ -172,5 +172,5 @@
     <!-- Camera -->
   <joint type="fixed" name="camera_joint">
-    <origin xyz="0.300 -0.005 0.075" rpy="0 0 0"/>
+    <origin xyz="0.350 -0.005 0.075" rpy="0 0 0"/>
     <child link="camera_link"/>
     <parent link="base_link"/>

Commit message: Acker initial
Not yet working, development in progress

File: line_follower_race_car/urdf/mogi_bot.xacro (robot description, xacro)
@@ -1,213 +1,138 @@
-<?xml version='1.0'?>
-<robot name="mogi_bot" xmlns:xacro="http://www.ros.org/wiki/xacro">
-  <!-- STEP 3 - Gazebo plugin -->
-  <xacro:include filename="$(find line_follower_race_car)/urdf/mogi_bot.gazebo" />
-  <!-- STEP 4 - RViz colors -->
-  <xacro:include filename="$(find line_follower_race_car)/urdf/materials.xacro" />
-  <!-- STEP 1 - Robot chassis -->
-  <link name="base_footprint"></link>
-  <joint name="base_footprint_joint" type="fixed">
-    <origin xyz="0 0 0" rpy="0 0 -1.5707" />
-    <parent link="base_footprint"/>
-    <child link="base_link" />
-  </joint>
-  <link name='base_link'>
-    <pose>0 0 0.1 0 0 0</pose>
-    <inertial>
-      <mass value="15.0"/>
-      <origin xyz="0.0 0 0" rpy=" 0 0 0"/>
-      <inertia
-          ixx="0.1" ixy="0" ixz="0"
-          iyy="0.1" iyz="0"
-          izz="0.1"
-      />
-    </inertial>
-    <collision name='collision'>
-      <origin xyz="0 0 0" rpy=" 0 0 -1.5707"/>
+<?xml version="1.0"?>
+<!--
+  Robot model adapted from https://github.com/CIR-KIT/steer_drive_ros/blob/kinetic-devel/steer_drive_controller/test/common/urdf/steerbot.xacro
+  Modifications:
+    Almost all...
+  Geometry:
+    The Ackermann steering controllers require the longitudinal
+    separation between the front and back wheel axes and the
+    lateral separation between the left and right front steering axes.
+    For this model:
+    wheel_separation_h = base_length - 2 * axle_offset = 0.4
+    wheel_separation_w = base_width  + 2 * axle_offset = 0.4
+-->
+<robot name="steer_bot" xmlns:xacro="http://wiki.ros.org/xacro">
+  <!-- Include xacro for inertials, materials and wheels -->
+  <xacro:include filename="$(find line_follower_race_car)/urdf/wheel.xacro"/>
+  <xacro:property name="robot_namespace" value="/line_follower_race_car"/>
+  <!-- Gazebo plugins -->
+  <gazebo>
+    <!-- Load ros_control plugin using the steer_bot_hardware_gazebo
+    implementation of the hardware_interface::RobotHW -->
+    <plugin name="gazebo_ros_control" filename="libgazebo_ros_control.so">
+      <robotNamespace>${robot_namespace}</robotNamespace>
+      <robotSimType>steer_bot_hardware_gazebo/SteerBotHardwareGazebo</robotSimType>
+      <legacyModeNS>false</legacyModeNS>
+    </plugin>
+  </gazebo>
+  <!-- Math constants -->
+  <xacro:property name="deg_to_rad" value="0.01745329251994329577"/>
+  <!-- Robot base dimensions -->
+  <xacro:property name="base_length" value="0.4" />
+  <xacro:property name="base_width" value="0.2" />
+  <xacro:property name="base_height" value="0.1" />
+  <xacro:property name="base_mass" value="15" />
+  <xacro:property name="base_rpy" value="0 0 -1.5707"
+  <!-- Wheel link dimensions -->
+  <xacro:property name="wheel_radius" value="0.1" />
+  <xacro:property name="wheel_thickness" value="0.08" />
+  <xacro:property name="wheel_mass" value="1" />
+  <!-- Steering link dimensions -->
+  <xacro:property name="steer_radius" value="0.05" />
+  <xacro:property name="steer_thickness" value="0.02" />
+  <xacro:property name="steer_mass" value="1" />
+  <!-- Axle positions -->
+  <xacro:property name="axle_offset" value="0.05" />
+  <xacro:property name="steer_offset" value="0.02" />
+  <!-- Base link -->
+  <link name="base_link">
+    <visual>
+      <origin xyz="0 0 0" rpy="${base_rpy}"/>
       <geometry>
-        <box size=".4 .2 .1"/>
-      </geometry>
-    </collision>
-    <visual name='base_link_visual'>
-      <origin xyz="0 0 0" rpy=" 0 0 -1.5707"/>
-      <geometry>
-        <!--box size=".4 .2 .1"/-->
         <mesh filename = "package://line_follower_race_car/meshes/body.dae"/>
       </geometry>
     </visual>
-  </link>
-  <!-- STEP 2 - Wheels -->
-  <!-- Front left -->
-  <joint type="continuous" name="front_left_wheel_joint">
-    <origin xyz="0.23 0.17 0" rpy="0 0 0"/>
-    <child link="front_left_wheel"/>
-    <parent link="base_link"/>
-    <axis xyz="0 1 0" rpy="0 0 0"/>
-    <limit effort="10000" velocity="1000"/>
-    <dynamics damping="1.0" friction="1.0"/>
-  </joint>
-  <link name='front_left_wheel'>
-    <inertial>
-      <mass value="5.0"/>
-      <origin xyz="0 0 0" rpy="0 1.5707 1.5707"/>
-      <inertia
-          ixx="0.1" ixy="0" ixz="0"
-          iyy="0.1" iyz="0"
-          izz="0.1"
-      />
-    </inertial>
-    <collision name='collision'>
-      <origin xyz="0 0 0" rpy="0 1.5707 1.5707"/>
+    <collision>
+      <origin xyz="0 0 0" rpy="${base_rpy}"/>
       <geometry>
-        <cylinder radius=".1" length=".05"/>
+        <box size="${base_length} ${base_width} ${base_height}"/>
       </geometry>
     </collision>
-    <visual name='front_left_wheel_visual'>
-      <origin xyz="0 0 0" rpy="0 1.5707 1.5707"/>
-      <geometry>
-        <!--cylinder radius=".1" length=".05"/-->
-        <mesh filename = "package://line_follower_race_car/meshes/front_wheels.dae"/>
-      </geometry>
-    </visual>
+    <xacro:solid_cuboid_inertial
+        rpy="${base_rpy}" xyz="0 0 0"
+        mass="${base_mass}"
+        x="${base_length}" y="${base_width}" z="${base_height}" />
   </link>
-<!-- Front right -->
-  <joint type="continuous" name="front_right_wheel_joint">
-    <origin xyz="0.23 -0.19 0" rpy="0 0 0"/>
-    <child link="front_right_wheel"/>
-    <parent link="base_link"/>
-    <axis xyz="0 1 0" rpy="0 0 0"/>
-    <limit effort="10000" velocity="1000"/>
-    <dynamics damping="1.0" friction="1.0"/>
-  </joint>
-  <link name='front_right_wheel'>
-    <inertial>
-      <mass value="5.0"/>
-      <origin xyz="0 0 0" rpy="0 1.5707 -1.5707"/>
-      <inertia
-          ixx="0.1" ixy="0" ixz="0"
-          iyy="0.1" iyz="0"
-          izz="0.1"
-      />
-    </inertial>
-    <collision name='collision'>
-      <origin xyz="0 0 0" rpy="0 1.5707 -1.5707"/>
-      <geometry>
-        <cylinder radius=".1" length=".05"/>
-      </geometry>
-    </collision>
-    <visual name='front_right_wheel_visual'>
-      <origin xyz="0 0 0" rpy="0 1.5707 -1.5707"/>
-      <geometry>
-        <!--cylinder radius=".1" length=".05"/-->
-        <mesh filename = "package://line_follower_race_car/meshes/front_wheels.dae"/>
-      </geometry>
-    </visual>
-  </link>
-<!-- Rear left -->
-  <joint type="continuous" name="rear_left_wheel_joint">
-    <origin xyz="-0.25 0.17 0" rpy="0 0 0"/>
-    <child link="rear_left_wheel"/>
-    <parent link="base_link"/>
-    <axis xyz="0 1 0" rpy="0 0 0"/>
-    <limit effort="10000" velocity="1000"/>
-    <dynamics damping="1.0" friction="1.0"/>
-  </joint>
-  <link name='rear_left_wheel'>
-    <inertial>
-      <mass value="5.0"/>
-      <origin xyz="0 0 0" rpy="0 1.5707 1.5707"/>
-      <inertia
-          ixx="0.1" ixy="0" ixz="0"
-          iyy="0.1" iyz="0"
-          izz="0.1"
-      />
-    </inertial>
-    <collision name='collision'>
-      <origin xyz="0 0 0" rpy="0 1.5707 1.5707"/>
-      <geometry>
-        <cylinder radius=".1" length=".05"/>
-      </geometry>
-    </collision>
-    <visual name='rear_left_wheel_visual'>
-      <origin xyz="0 0 0" rpy="0 1.5707 1.5707"/>
-      <geometry>
-        <!--cylinder radius=".1" length=".05"/-->
-        <mesh filename = "package://line_follower_race_car/meshes/front_wheels.dae"/>
-      </geometry>
-    </visual>
-  </link>
-<!-- Rear right -->
-  <joint type="continuous" name="rear_right_wheel_joint">
-    <origin xyz="-0.25 -0.19 0" rpy="0 0 0"/>
-    <child link="rear_right_wheel"/>
-    <parent link="base_link"/>
-    <axis xyz="0 1 0" rpy="0 0 0"/>
-    <limit effort="10000" velocity="1000"/>
-    <dynamics damping="1.0" friction="1.0"/>
-  </joint>
-  <link name='rear_right_wheel'>
-    <inertial>
-      <mass value="5.0"/>
-      <origin xyz="0 0 0" rpy="0 1.5707 -1.5707"/>
-      <inertia
-          ixx="0.1" ixy="0" ixz="0"
-          iyy="0.1" iyz="0"
-          izz="0.1"
-      />
-    </inertial>
-    <collision name='collision'>
-      <origin xyz="0 0 0" rpy="0 1.5707 -1.5707"/>
-      <geometry>
-        <cylinder radius=".1" length=".05"/>
-      </geometry>
-    </collision>
-    <visual name='rear_right_wheel_visual'>
-      <origin xyz="0 0 0" rpy="0 1.5707 -1.5707"/>
-      <geometry>
-        <!--cylinder radius=".1" length=".05"/-->
-        <mesh filename = "package://line_follower_race_car/meshes/front_wheels.dae"/>
-      </geometry>
-    </visual>
-  </link>
-    <!-- Camera -->
-  <joint type="fixed" name="camera_joint">
-    <origin xyz="0.300 -0.005 0.075" rpy="0 0 0"/>
-    <child link="camera_link"/>
-    <parent link="base_link"/>
-    <axis xyz="0 1 0" />
-  </joint>
-  <link name='camera_link'>
-    <pose>0 0 0 0 0 0</pose>
-    <inertial>
-      <mass value="0.1"/>
-      <origin xyz="0 0 0" rpy="0 0 0"/>
-      <inertia
-          ixx="1e-6" ixy="0" ixz="0"
-          iyy="1e-6" iyz="0"
-          izz="1e-6"
-      />
-    </inertial>
-    <collision name='collision'>
-      <origin xyz="0 0 0" rpy="0 0 0"/>
-      <geometry>
-        <box size=".05 .05 .05"/>
-      </geometry>
-    </collision>
-    <visual name='camera_link_visual'>
-      <origin xyz="0 0 0" rpy="0 0 0"/>
-      <geometry>
-        <box size=".05 .05 .05"/>
-      </geometry>
-    </visual>
-  </link>
-  <gazebo reference="camera_link">
-    <material>Gazebo/Red</material>
+  <!-- Front steer and rear wheel joints required for ackermann_steering_controller -->
+  <xacro:front_steer
+    name="front"
+    parent="base"
+    steer_radius="${steer_radius}"
+    steer_thickness="${steer_thickness}"
+    steer_mass="${steer_mass}"
+    base_length="${base_length}"
+    base_width="${base_width}"
+    axle_offset="${axle_offset}"
+    steer_height="${wheel_radius+steer_offset}">
+  </xacro:front_steer>
+  <xacro:rear_wheel
+    name="rear"
+    parent="base"
+    wheel_radius="${wheel_radius/4}"
+    wheel_thickness="${wheel_thickness/2}"
+    wheel_mass="${wheel_mass/32}">
+    <origin xyz="${-base_length/2+axle_offset} 0 0" rpy="${-90 * deg_to_rad} 0 0"/>
+  </xacro:rear_wheel>
+  <!-- Steerable front wheels -->
+  <xacro:front_wheel_lr
+    name="front_right"
+    parent="base"
+    reflect="-1"
+    wheel_radius="${wheel_radius}"
+    wheel_thickness="${wheel_thickness}"
+    wheel_mass="${wheel_mass}"
+    steer_radius="${steer_radius}"
+    steer_thickness="${steer_thickness}"
+    steer_mass="${steer_mass}"
+    base_length="${base_length}"
+    base_width="${base_width}"
+    axle_offset="${axle_offset}"
+    steer_height="${wheel_radius+steer_offset}">
+  </xacro:front_wheel_lr>
+  <xacro:front_wheel_lr
+    name="front_left"
+    parent="base"
+    reflect="1"
+    wheel_radius="${wheel_radius}"
+    wheel_thickness="${wheel_thickness}"
+    wheel_mass="${wheel_mass}"
+    steer_radius="${steer_radius}"
+    steer_thickness="${steer_thickness}"
+    steer_mass="${steer_mass}"
+    base_length="${base_length}"
+    base_width="${base_width}"
+    axle_offset="${axle_offset}"
+    steer_height="${wheel_radius+steer_offset}">
+  </xacro:front_wheel_lr>
+  <!-- Rear wheels -->
+  <xacro:rear_wheel_lr
+    name="rear_right"
+    parent="base"
+    wheel_radius="${wheel_radius}"
+    wheel_thickness="${wheel_thickness}"
+    wheel_mass="${wheel_mass}">
+    <origin xyz="${-base_length/2+axle_offset} ${-base_width/2-axle_offset} 0" rpy="${-90 * deg_to_rad} 0 0"/>
+  </xacro:rear_wheel_lr>
+  <xacro:rear_wheel_lr
+    name="rear_left"
+    parent="base"
+    wheel_radius="${wheel_radius}"
+    wheel_thickness="${wheel_thickness}"
+    wheel_mass="${wheel_mass}">
+    <origin xyz="${-base_length/2+axle_offset} ${+base_width/2+axle_offset} 0" rpy="${-90 * deg_to_rad} 0 0"/>
+  </xacro:rear_wheel_lr>
+  <!-- Colour -->
+  <gazebo reference="base_link">
+    <material>Gazebo/Green</material>
   </gazebo>
-  <joint type="fixed" name="camera_optical_joint">
-    <origin xyz="0 0 0" rpy="-1.5707 0 -1.5707"/>
-    <child link="camera_link_optical"/>
-    <parent link="camera_link"/>
-  </joint>
-  <link name="camera_link_optical">
-  </link>
 </robot>
