Commit message: Dead end
Too complicated, not gonna work

File: line_follower_race_car/urdf/mogi_bot.xacro (robot description, xacro)
@@ -15,5 +15,4 @@
   <!-- Include xacro for inertials, materials and wheels -->
   <xacro:include filename="$(find line_follower_race_car)/urdf/wheel.xacro"/>
-  <xacro:property name="robot_namespace" value="/line_follower_race_car"/>
   <!-- Gazebo plugins -->
   <gazebo>
@@ -21,7 +20,5 @@
     implementation of the hardware_interface::RobotHW -->
     <plugin name="gazebo_ros_control" filename="libgazebo_ros_control.so">
-      <robotNamespace>${robot_namespace}</robotNamespace>
       <robotSimType>steer_bot_hardware_gazebo/SteerBotHardwareGazebo</robotSimType>
-      <legacyModeNS>true</legacyModeNS>
     </plugin>
   </gazebo>

Commit message: Track following done.

File: line_follower_race_car/urdf/mogi_bot.xacro (robot description, xacro)
@@ -13,8 +13,8 @@
   </joint>
   <link name='base_link'>
-    <pose>0 0 0.1 0 0 0</pose>
+    <pose>0 0 0.1 0 0 -1.5707</pose>
     <inertial>
       <mass value="15.0"/>
-      <origin xyz="0.0 0 0" rpy=" 0 0 0"/>
+      <origin xyz="0.0 0 0" rpy="0 0 0"/>
       <inertia
           ixx="0.1" ixy="0" ixz="0"
@@ -172,5 +172,5 @@
     <!-- Camera -->
   <joint type="fixed" name="camera_joint">
-    <origin xyz="0.350 -0.005 0.075" rpy="0 0 0"/>
+    <origin xyz="0.350 -0.005 0.075" rpy="0 0.785 0"/>
     <child link="camera_link"/>
     <parent link="base_link"/>
